File: common_parts_library.sch (KiCad schematic (older format))
At the start: 10 parts

Commit message: Schematic Symbol Update 09-NOV-2014
Completed schematic symbols for resistors, capacitors, inductors, LEDs,
Diodes and Transistors.
Parts:
- removed D?: D_CPL, ~, symbol D_CPL
- removed D?: LED_CPL, ~, symbol LED_CPL
- removed Q?: NPN_CPL, symbol NPN_CPL
- removed Q?: PNP_CPL, symbol PNP_CPL
- removed Q?: PNP_DUAL_CPL, ~, symbol PNP_DUAL_CPL
- added D?: D_SCHOTTKY_CPL, ~, symbol D_SCHOTTKY_CPL
- added D? (x2): D_SCHOTTKY_BAT54S_CPL, ~, symbol D_SCHOTTKY_BAT54S_CPL
- added D? (x2): D_SCHOTTKY_BAS70-04_CPL, ~, symbol D_SCHOTTKY_BAS70-04_CPL
- added D?: LED_CPL, ~, symbol LED_CPL
- added D?: D_CPL, ~, symbol D_CPL
- added D?: D_PINSWAP_CPL, ~, symbol D_PINSWAP_CPL
- added LED?: LED_RGB_WS2812_CPL, symbol LED_RGB_WS2812_CPL
- added Q?: NPN_CPL, ~, symbol NPN_CPL
- added Q?: PNP_CPL, ~, symbol PNP_CPL
- added Q?: PNP_DUAL_CPL, ~, symbol PNP_DUAL_CPL
- added Q?: PNP_DUAL_PINSWAP_CPL, ~, symbol PNP_DUAL_PINSWAP_CPL
- added Q?: N_CHANNEL_FET_CPL, ~, symbol N_CHANNEL_FET_CPL
- added Q?: P_CHANNEL_FET_CPL, ~, symbol P_CHANNEL_FET_CPL
- added Q?: N_CHANNEL_POWER_MOSFET_CPL, ~, symbol N_CHANNEL_POWER_MOSFET_CPL
- added R?: POTENTIOMETER_CPL, ~, symbol POTENTIOMETER_CPL
Other:
- moved on the sheet: C?, L?, R?
